Commit message: fix

File: src/rosiwit_simulator/urdf/xacro/gazebo/mbot_with_lidar3d_gazebo.xacro (robot description, xacro)
@@ -9,5 +9,5 @@
     <xacro:include filename="$(find rosiwit_simulator)/urdf/xacro/sensors/lidar3d_gazebo.xacro" />
     <xacro:include filename="$(find rosiwit_simulator)/urdf/xacro/sensors/imu_gazebo.xacro" />
-    <xacro:lidar3d_gazebo prefix="velodyne"/>
+    <xacro:lidar3d_gazebo prefix="lidar"/>
     <xacro:imu prefix="imu"/>
     <xacro:mbot_base/>

File: src/rosiwit_simulator/urdf/xacro/sensors/lidar3d.xacro (robot description, xacro)
@@ -5,5 +5,5 @@
         Defines link/joint only, no Gazebo plugin (see lidar3d_gazebo.xacro)
     -->
-    <xacro:macro name="lidar3d" params="prefix:=velodyne">
+    <xacro:macro name="lidar3d" params="prefix:=lidar">
         <!-- VLP-16: radius=0.0516m, height=0.0717m -->
         <link name="${prefix}_link">

File: src/rosiwit_simulator/urdf/xacro/sensors/lidar3d_gazebo.xacro (robot description, xacro)
@@ -9,5 +9,5 @@
         - frameName: velodyne_link  (must match URDF link name for TF consistency)
     -->
-    <xacro:macro name="lidar3d_gazebo" params="prefix:=velodyne">
+    <xacro:macro name="lidar3d_gazebo" params="prefix:=lidar">
         <!-- Include physical description from lidar3d.xacro -->
         <xacro:include filename="$(find rosiwit_simulator)/urdf/xacro/sensors/lidar3d.xacro" />
@@ -50,5 +50,5 @@
                     </ros>
                     <output_type>sensor_msgs/PointCloud2</output_type>
-                    <frame_name>velodyne_link</frame_name>
+                    <frame_name>lidar_link</frame_name>
                 </plugin>
             </sensor>
