Commit message: fix

File: src/rosiwit_simulator/urdf/xacro/gazebo/mbot_with_fisheye_gazebo.xacro (robot description, xacro)
@@ -8,5 +8,5 @@
     <xacro:imu prefix="imu"/>
     <xacro:rplidar prefix="laser"/>
-    <xacro:lidar3d_gazebo prefix="velodyne"/>
+    <xacro:lidar3d_gazebo prefix="lidar"/>
     <!-- 4 个广角相机，90°间隔，360°全覆盖，向下倾斜 20° 看到地面 -->
     <!-- 位置：底座半径 0.21m，高出底座 0.15m -->

File: src/rosiwit_simulator/urdf/xacro/sensors/lidar_gazebo.xacro (robot description, xacro)
@@ -29,5 +29,5 @@
         </link>
         <!-- Create laser joint-->
-        <joint name="lidar_joint" type="fixed">
+        <joint name="laser_joint" type="fixed">
             <origin xyz="${lidar_offset_x} ${lidar_offset_y} ${lidar_offset_z}" rpy="0 0 0" />
             <parent link="base_link"/>
