Commit message: feat(ros1): GT 实机模型仿真 (3D+2D 雷达) + 定位/导航对齐实车
仿真 (rosiwit_simulation_ros1):
- GT 整车模型 (gt.glb -> gt.dae 单网格), 按实车 xzrobot.v3.urdf 复刻
  传感器/坐标架; 模型原点前移 0.119 对齐驱动轮轴, 车头与前声呐对齐
- 车体碰撞体改为 0.87x0.70 长方体 (上下两块, 在 2D 雷达平面留缝)
- 新增实机 2D 雷达 Vanjee 716N: /scan, frame laser, +-2.18rad,
  1000 点, 0.1..30m, 15Hz, 安装位与实车一致 (0.47,0,0.115)
- 3D 雷达自带 velodyne 插件 (10Hz, 240x32), 机身自过滤/倾斜安装

导航 (rosiwit_navigation_ros1):
- footprint / robot_radius / inflation / 停障-减速多边形 / 速度限制
  全部对齐实车 default.yaml (footprint x -0.25..0.55, y +-0.33)
- require_scan=true, 安全层启用, scan 自滤盒用实车值
- MPPI + footprint 采样, AsyncSpinner, 诊断定时器发布 /robot_footprint

SLAM (rosiwit_slam_ros1 / rosiwit_slam):
- 定位模式点云输出应用 r_il/t_il 外参 (倾斜雷达不再用原始雷达系点云)
- 无逐点时间戳时可按方位角推导逐点时间 (scan_period_ms 开关, 仿真默认关)
- 修复 Sophus 非正交崩溃 (ieskf/fast_lio2/point_lio)
- 建图 PCD->栅格重建工具, 保存地图加载 (load_saved_map)

其它:
- 新增 rosiwit_starter_ros1 一键仿真 (slam_simulation / navigation_simulation)
- 仿真地图 docs/maps/house_sim (gitignore), 实车地图 docs/maps/map

File: ros1_ws/src/rosiwit_simulation_ros1/urdf/xacro/gazebo/mbot_base.xacro (robot description, xacro)
@@ -40,5 +40,5 @@
     </xacro:macro>
     <!-- Macro for robot wheel -->
-    <xacro:macro name="wheel" params="prefix reflect">
+    <xacro:macro name="wheel" params="prefix reflect show_visual:=1">
         <joint name="${prefix}_wheel_joint" type="continuous">
             <origin xyz="0 ${reflect*wheel_joint_y} ${-wheel_joint_z}" rpy="0 0 0"/>
@@ -48,4 +48,5 @@
         </joint>
         <link name="${prefix}_wheel_link">
+            <xacro:if value="${int(show_visual) == 1}">
             <visual>
                 <origin xyz="0 0 0" rpy="${M_PI/2} 0 0" />
@@ -55,4 +56,5 @@
                 <material name="gray" />
             </visual>
+            </xacro:if>
             <collision>
                 <origin xyz="0 0 0" rpy="${M_PI/2} 0 0" />
@@ -79,5 +81,5 @@
     </xacro:macro>
     <!-- Macro for robot caster -->
-    <xacro:macro name="caster" params="prefix reflect">
+    <xacro:macro name="caster" params="prefix reflect show_visual:=1">
         <joint name="${prefix}_caster_joint" type="continuous">
             <origin xyz="${reflect*caster_joint_x} 0 ${-(base_length/2 + caster_radius)}" rpy="0 0 0"/>
@@ -87,4 +89,5 @@
         </joint>
         <link name="${prefix}_caster_link">
+            <xacro:if value="${int(show_visual) == 1}">
             <visual>
                 <origin xyz="0 0 0" rpy="0 0 0"/>
@@ -94,4 +97,5 @@
                 <material name="black" />
             </visual>
+            </xacro:if>
             <collision>
                 <origin xyz="0 0 0" rpy="0 0 0"/>
@@ -106,6 +110,7 @@
         </gazebo>
     </xacro:macro>
-    <xacro:macro name="mbot_base">
+    <xacro:macro name="mbot_base" params="show_visual:=1 base_mesh:='' base_mesh_xyz:='0 0 0' base_mesh_rpy:='0 0 0' base_collision_box:='' base_collision_xyz:='0 0 0' base_collision_box2:='' base_collision_xyz2:='0 0 0'">
         <link name="base_footprint">
+            <xacro:if value="${int(show_visual) == 1}">
             <visual>
                 <origin xyz="0 0 0" rpy="0 0 0" />
@@ -114,4 +119,5 @@
                 </geometry>
             </visual>
+            </xacro:if>
         </link>
         <gazebo reference="base_footprint">
@@ -124,4 +130,5 @@
         </joint>
         <link name="base_link">
+            <xacro:if value="${int(show_visual) == 1}">
             <visual>
                 <origin xyz=" 0 0 0" rpy="0 0 0" />
@@ -131,9 +138,36 @@
                 <material name="yellow" />
             </visual>
+            </xacro:if>
+            <!-- 可选: 用外来整车网格替换默认圆柱外观 (实机模型) -->
+            <xacro:unless value="${base_mesh == ''}">
+                <visual>
+                    <origin xyz="${base_mesh_xyz}" rpy="${base_mesh_rpy}" />
+                    <geometry>
+                        <mesh filename="${base_mesh}" scale="1 1 1"/>
+                    </geometry>
+                </visual>
+            </xacro:unless>
             <collision>
-                <origin xyz=" 0 0 0" rpy="0 0 0" />
-                <geometry>
-                    <cylinder length="${base_length}" radius="${base_radius}"/>
-                </geometry>
+                <xacro:if value="${base_collision_box != ''}">
+                    <!-- box collision that matches the real chassis outline -->
+                    <origin xyz="${base_collision_xyz}" rpy="0 0 0" />
+                    <geometry>
+                        <box size="${base_collision_box}"/>
+                    </geometry>
+                </xacro:if>
+                <xacro:if value="${base_collision_box2 != ''}">
+                    <!-- second box: leave a gap at the 2D lidar plane so the
+                         ray sensor can see out of the chassis -->
+                    <origin xyz="${base_collision_xyz2}" rpy="0 0 0" />
+                    <geometry>
+                        <box size="${base_collision_box2}"/>
+                    </geometry>
+                </xacro:if>
+                <xacro:unless value="${base_collision_box != ''}">
+                    <origin xyz=" 0 0 0" rpy="0 0 0" />
+                    <geometry>
+                        <cylinder length="${base_length}" radius="${base_radius}"/>
+                    </geometry>
+                </xacro:unless>
             </collision>
             <xacro:cylinder_inertial_matrix  m="${base_mass}" r="${base_radius}" h="${base_length}" />
@@ -142,8 +176,8 @@
             <material>Gazebo/Blue</material>
         </gazebo>
-        <xacro:wheel prefix="left"  reflect="1"/>
-        <xacro:wheel prefix="right" reflect="-1"/>
-        <xacro:caster prefix="front" reflect="-1"/>
-        <xacro:caster prefix="back"  reflect="1"/>
+        <xacro:wheel prefix="left"  reflect="1"  show_visual="${show_visual}"/>
+        <xacro:wheel prefix="right" reflect="-1" show_visual="${show_visual}"/>
+        <xacro:caster prefix="front" reflect="-1" show_visual="${show_visual}"/>
+        <xacro:caster prefix="back"  reflect="1"  show_visual="${show_visual}"/>
         <!-- controller (ROS1 gazebo_ros_diff_drive) -->
         <gazebo>

File: ros1_ws/src/rosiwit_simulation_ros1/urdf/xacro/gazebo/mbot_with_lidar3d_gazebo.xacro (robot description, xacro)
@@ -9,5 +9,10 @@
     <xacro:include filename="$(find rosiwit_simulation_ros1)/urdf/xacro/sensors/lidar3d_gazebo.xacro" />
     <xacro:include filename="$(find rosiwit_simulation_ros1)/urdf/xacro/sensors/imu_gazebo.xacro" />
-    <xacro:lidar3d_gazebo prefix="lidar"/>
+    <!-- lidar_plugin: block (default, gazebo_plugins built-in) | velodyne
+         velodyne needs ros-melodic-velodyne-gazebo-plugins for a more faithful
+         VLP-16 cloud; both publish on the same topic/frame.
+         Keep this file ASCII-only (Python 2 URDF parsers). -->
+    <xacro:arg name="lidar_plugin" default="block"/>
+    <xacro:lidar3d_gazebo prefix="lidar" plugin="$(arg lidar_plugin)"/>
     <xacro:imu prefix="imu"/>
     <xacro:mbot_base/>

File: ros1_ws/src/rosiwit_simulation_ros1/urdf/xacro/sensors/imu_gazebo.xacro (robot description, xacro)
@@ -1,8 +1,5 @@
 <?xml version="1.0"?>
 <robot xmlns:xacro="http://www.ros.org/wiki/xacro" name="imu">
-    <xacro:macro name="imu" params="prefix:=imu">
-        <xacro:property name="imu_offset_x" value="0" />
-        <xacro:property name="imu_offset_y" value="0" />
-        <xacro:property name="imu_offset_z" value="0.105" />
+    <xacro:macro name="imu" params="prefix:=imu offset_x:=0 offset_y:=0 offset_z:=0.105 offset_rpy:='0 0 0'">
         <link name="${prefix}_link">
             <inertial>
@@ -28,5 +25,5 @@
         </link>
         <joint name="imu_joint" type="fixed">
-            <origin xyz="${imu_offset_x} ${imu_offset_y} ${imu_offset_z}" rpy="0 0 0" />
+            <origin xyz="${offset_x} ${offset_y} ${offset_z}" rpy="${offset_rpy}" />
             <parent link="base_link"/>
             <child link="imu_link"/>

File: ros1_ws/src/rosiwit_simulation_ros1/urdf/xacro/sensors/lidar3d.xacro (robot description, xacro)
@@ -5,7 +5,8 @@
         Defines link/joint only, no Gazebo plugin (see lidar3d_gazebo.xacro)
     -->
-    <xacro:macro name="lidar3d" params="prefix:=lidar">
+    <xacro:macro name="lidar3d" params="prefix:=lidar mount_x:=0 mount_y:=0 mount_z:=0.1955 mount_rpy:='0 0 0'">
         <!-- VLP-16: radius=0.0516m, height=0.0717m -->
-        <link name="${prefix}_link">
+        <!-- The real robot names this link "lidar" (xzrobot.v3.urdf) -->
+        <link name="${prefix}">
             <inertial>
                 <mass value="0.83" />
@@ -38,9 +39,9 @@
              (matches architecture spec) -->
         <joint name="${prefix}_joint" type="fixed">
-            <origin xyz="0 0 0.1955" rpy="0 0 0" />
+            <origin xyz="${mount_x} ${mount_y} ${mount_z}" rpy="${mount_rpy}" />
             <parent link="base_link"/>
-            <child link="${prefix}_link"/>
+            <child link="${prefix}"/>
         </joint>
-        <gazebo reference="${prefix}_link">
+        <gazebo reference="${prefix}">
             <material>Gazebo/Grey</material>
         </gazebo>

File: ros1_ws/src/rosiwit_simulation_ros1/urdf/xacro/sensors/lidar3d_gazebo.xacro (robot description, xacro)
@@ -2,15 +2,25 @@
 <robot xmlns:xacro="http://www.ros.org/wiki/xacro" name="lidar3d">
     <!--
-        3D LiDAR Gazebo plugin configuration (ROS1)
+        3D LiDAR Gazebo plugin configuration (ROS1).
         Simulates a Velodyne VLP-16 and publishes sensor_msgs/PointCloud2
         on /velodyne_points.
-        Uses velodyne_gazebo_plugins (ROS1 Melodic/Noetic), which is the
-        drop-in 3D ray plugin for ROS1. (Noetic also ships
-        libgazebo_ros_ray_sensor.so, but Melodic does not.)
+        Two plugin backends, selected by the xacro arg "lidar_plugin":
+          block    (default) libgazebo_ros_block_laser.so from gazebo_plugins.
+                   Works with a minimal melodic install, but publishes the
+                   legacy sensor_msgs/PointCloud, so pointcloud_relay converts
+                   /velodyne_points_raw into /velodyne_points (PointCloud2).
+          velodyne libgazebo_ros_velodyne_laser.so from
+                   velodyne_gazebo_plugins (apt: ros-melodic-velodyne-gazebo-plugins).
+                   Publishes PointCloud2 directly, closer to a real VLP-16.
+        Both use the same <sensor type="ray"> and the same output topic/frame,
+        so SLAM and navigation do not need to care which one is active.
+        NOTE: keep this file ASCII-only. Python 2 tools (spawn_model,
+        joint_state_publisher) parse the expanded URDF as ASCII and fail on
+        non-ASCII bytes in comments.
     -->
-    <xacro:macro name="lidar3d_gazebo" params="prefix:=lidar">
+    <xacro:macro name="lidar3d_gazebo" params="prefix:=lidar plugin:=block mount_x:=0 mount_y:=0 mount_z:=0.1955 mount_rpy:='0 0 0'">
         <xacro:include filename="$(find rosiwit_simulation_ros1)/urdf/xacro/sensors/lidar3d.xacro" />
-        <xacro:lidar3d prefix="${prefix}" />
-        <gazebo reference="${prefix}_link">
+        <xacro:lidar3d prefix="${prefix}" mount_x="${mount_x}" mount_y="${mount_y}" mount_z="${mount_z}" mount_rpy="${mount_rpy}" />
+        <gazebo reference="${prefix}">
             <sensor type="ray" name="velodyne_vlp16">
                 <pose>0 0 0 0 0 0</pose>
@@ -18,7 +28,12 @@
                 <update_rate>10</update_rate>
                 <ray>
+                    <!-- Aligned with the real 3D lidar on 192.168.21.166
+                         (/vanjee_points722): 32 lines, 360 deg, 10 Hz, vertical FOV
+                         -11.8 .. +50.7 deg in the lidar frame. The real mount is pitched
+                         43 deg + yawed 90 deg; with a 16-line +-15 deg sensor the tilted
+                         scan almost only sees the floor and FastLIO drifts. -->
                     <scan>
                         <horizontal>
-                            <samples>900</samples>
+                            <samples>240</samples>
                             <resolution>1</resolution>
                             <min_angle>-3.14159</min_angle>
@@ -26,13 +41,13 @@
                         </horizontal>
                         <vertical>
-                            <samples>16</samples>
+                            <samples>32</samples>
                             <resolution>1</resolution>
-                            <min_angle>-0.2618</min_angle>
-                            <max_angle>0.2618</max_angle>
+                            <min_angle>-0.20595</min_angle>
+                            <max_angle>0.88487</max_angle>
                         </vertical>
                     </scan>
                     <range>
                         <min>0.10</min>
-                        <max>100.0</max>
+                        <max>30.0</max>
                         <resolution>0.01</resolution>
                     </range>
@@ -43,12 +58,22 @@
                     </noise>
                 </ray>
-                <plugin name="gazebo_ros_laser_controller" filename="libgazebo_ros_velodyne_laser.so">
-                    <topicName>velodyne_points</topicName>
-                    <frameName>lidar_link</frameName>
-                    <organize_cloud>false</organize_cloud>
-                    <min_range>0.10</min_range>
-                    <max_range>100.0</max_range>
-                    <gaussianNoise>0.01</gaussianNoise>
-                </plugin>
+                <xacro:if value="${plugin == 'velodyne'}">
+                    <plugin name="gazebo_ros_laser_controller" filename="libgazebo_ros_velodyne_laser.so">
+                        <topicName>velodyne_points</topicName>
+                        <frameName>${prefix}</frameName>
+                        <organize_cloud>false</organize_cloud>
+                        <min_range>0.10</min_range>
+                        <max_range>100.0</max_range>
+                        <gaussianNoise>0.01</gaussianNoise>
+                    </plugin>
+                </xacro:if>
+                <xacro:unless value="${plugin == 'velodyne'}">
+                    <plugin name="gazebo_ros_block_laser" filename="libgazebo_ros_block_laser.so">
+                        <!-- legacy PointCloud -> relay -> PointCloud2 -->
+                        <topicName>velodyne_points_raw</topicName>
+                        <frameName>${prefix}</frameName>
+                        <gaussianNoise>0.01</gaussianNoise>
+                    </plugin>
+                </xacro:unless>
             </sensor>
         </gazebo>
